File: hardware/kicad/matrix.kicad_sch (KiCad schematic)
At the start: 24 parts, among them U3 PGA2310PA, U4 PGA2310PA, U5 OPA2134PA

Commit message: Rev C: XIAO RP2040 and Traco TBA 2-0522 replace the Teensy 4.0 and TMR 3
Tier 1 cost-down, no change to the audio path. U9 becomes a Seeed XIAO
RP2040 on header pins (USB-C, TinyUSB MIDI, its 5V pin is VBUS straight
through), PS1 becomes a 2 W unregulated Traco TBA 2-0522 on KiCad's stock
SIP-7 footprint. Rails are now +/-12 V: the +/-15 V TBA 2-0523 would pass
the PGA2310's 16 V absolute maximum at light load. Parts cost drops from
about $145 to about $110.

- gen.py: TBA2_Dual and XIAO_RP2040 symbols, XIAO footprint (Seeed pin
  numbering, USB-C overhang drawn), control sheet rewired to D0-D10,
  power sheet and notes for the unregulated converter, +/-12V rails.
- check.py: new U9 / PS1 pins; NETLIST OK. ERC 0/0.
- Both boards rebuilt and re-routed (Freerouting 1.9), DRC 0 errors; the
  only warnings are jack-nose and USB-C shell silk over the board edge.
- Gerbers, drill, zips, BOM, schematic SVG/PDF and board renders
  regenerated. README and site updated: pin map, power budget
  (~250 mA typical), level budget at +/-12 V, parts list and totals.

Co-Authored-By: Claude Fable 5.1 <noreply@anthropic.com>
Claude-Session: https://claude.ai/code/session_01C8uqpe49go1TPWMsWKKVkn
Connections:
- net +15V renamed +12V
- net -15V renamed -12V
Other:
- note added: "U3 = direct paths (L->L on its left channel, R->R on its right). U4 = cross paths (L->R on its left channel, R->L on its right). SPI chain: XIAO MOSI (D10) -> U3 SDI, U3 SDO -> U4 SDI. 32 clocks per update: U4 word first, then U3; each word is right byte then left byte, MSB first. ZCEN high: gain changes wait for a zero crossing. Code 192 = 0 dB, 0 = mute. Never route SDO (5 V logic) back to the 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"
- note removed: "U3 = direct paths (L->L on its left channel, R->R on its right). U4 = cross paths (L->R on its left channel, R->L on its right). SPI chain: Teensy MOSI -> U3 SDI, U3 SDO -> U4 SDI. 32 clocks per update: U4 word first, then U3; each word is right byte then left byte, MSB first. ZCEN high: gain changes wait for a zero crossing. Code 192 = 0 dB, 0 = mute. Never route SDO (5 V logic) back to the Teen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"

Commit message: Rev D: isolate the audio ground from USB
Add a TI ISO7762FDW digital isolator on the four control lines and two
plug-sense lines, a 78L05 that makes +5VA from +12 V for the PGA logic
and the isolator's audio side, and a split ground: GND_USB (XIAO, USB-C,
switch, LED, ferrite, reservoir, DC-DC input) and GND (everything audio).
The two meet only through C45 (1 nF) and R17 (1 M) at PS1. The sense
pull-ups drop from 1 M to 100 k for the isolator's input leakage.

Both boards get two ground pours per layer with a 2 mm copper-free gap
and a rule area that keeps the router out; U8 and PS1 straddle the gap.
The 1590BB board's island is the front-left corner; the narrow board's
is a pocket under the XIAO with the audio ground wrapping beneath it.
ERC 0, netlist checked (61 nets, 263 pins), DRC clean on both routed
boards, and a script check confirms no copper crosses the gap.

README, docs page, schematic exports, renders, gerbers and BOM regenerated.

Co-Authored-By: Claude Fable 5.1 <noreply@anthropic.com>
Claude-Session: https://claude.ai/code/session_013C8baRPktSQjwfdzSRwmAq
Connections:
- net +5V renamed +5VA
Other:
- note added: "Bypass, one per supply pin: U3 / U4 VA+, VA-, VD+; U5 V+, V-. C14 bulk on the +5VA logic rail beside U3."
- note added: "U3 = direct paths (L->L on its left channel, R->R on its right). U4 = cross paths (L->R on its left channel, R->L on its right). SPI chain: XIAO MOSI (D10) -> U8 isolator -> U3 SDI, U3 SDO -> U4 SDI. 32 clocks per update: U4 word first, then U3; each word is right byte then left byte, MSB first. ZCEN high: gain changes wait for a zero crossing. Code 192 = 0 dB, 0 = mute. Logic supply is +5VA from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"
- note removed: "Bypass, one per supply pin: U3 / U4 VA+, VA-, VD+; U5 V+, V-. C14 bulk on the 5 V logic rail beside U3."
- note removed: "U3 = direct paths (L->L on its left channel, R->R on its right). U4 = cross paths (L->R on its left channel, R->L on its right). SPI chain: XIAO MOSI (D10) -> U3 SDI, U3 SDO -> U4 SDI. 32 clocks per update: U4 word first, then U3; each word is right byte then left byte, MSB first. ZCEN high: gain changes wait for a zero crossing. Code 192 = 0 dB, 0 = mute. Never route SDO (5 V logic) back to the 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"
