File: hardware/kicad/output.kicad_sch (KiCad schematic)
At the start: 22 parts, among them J3 NRJ6HF, J4 NRJ6HF, U6 THAT1646S08, U7 THAT1646S08

Commit message: Add routed PCB layout, gerbers and PCB section on the site
- ghost-fader.kicad_pcb: 2-layer 108 x 80 mm board for the Hammond 1590BB,
  corner notches for the lid-screw bosses, jacks on the rear edge, Teensy USB
  flush with the front edge, DC-DC front-centre. Ground pour both layers,
  0.6 mm power / 0.3 mm signal tracks. DRC clean with schematic parity.
- tools/build_pcb.py (placement table, outline, pours, rules) and
  tools/route.py (Freerouting DSN/SES round trip) to regenerate the board.
- Jacks assigned KiCad's stock Neutrik NRJ6HF footprint; BOM regenerated.
- Design rules and Power net class in the project file and gen.py.
- Gerbers, drill and drill map in hardware/gerbers plus a zip for upload.
- Renders in docs/pcb and a PCB layout section on the published page;
  README PCB section.

Co-Authored-By: Claude Fable 5.1 <noreply@anthropic.com>
Claude-Session: https://claude.ai/code/session_015P372fhz9Ee8MTRWGXMeho
Parts:
- J3, J4: footprint (none) -> Connector_Audio:Jack_6.35mm_Neutrik_NRJ6HF_Horizontal
Changed lines of the file:
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@@
   (property "Reference" "J3" (at 154.94 39.37 0) (effects (font (size 1.27 1.27)) (justify left)))
   (property "Value" "NRJ6HF" (at 154.94 55.88 0) (effects (font (size 1.27 1.27)) (justify left)))
-  (property "Footprint" "" (at 157.48 50.8 0) (effects (font (size 1.27 1.27)) (hide yes)))
+  (property "Footprint" "Connector_Audio:Jack_6.35mm_Neutrik_NRJ6HF_Horizontal" (at 157.48 50.8 0) (effects (font (size 1.27 1.27)) (hide yes)))
   (property "Datasheet" "" (at 157.48 50.8 0) (effects (font (size 1.27 1.27)) (hide yes)))
   (pin "R")
@@
   (property "Reference" "J4" (at 154.94 100.33 0) (effects (font (size 1.27 1.27)) (justify left)))
   (property "Value" "NRJ6HF" (at 154.94 116.84 0) (effects (font (size 1.27 1.27)) (justify left)))
-  (property "Footprint" "" (at 157.48 111.76 0) (effects (font (size 1.27 1.27)) (hide yes)))
+  (property "Footprint" "Connector_Audio:Jack_6.35mm_Neutrik_NRJ6HF_Horizontal" (at 157.48 111.76 0) (effects (font (size 1.27 1.27)) (hide yes)))
   (property "Datasheet" "" (at 157.48 111.76 0) (effects (font (size 1.27 1.27)) (hide yes)))
   (pin "R")

Commit message: Rev C: XIAO RP2040 and Traco TBA 2-0522 replace the Teensy 4.0 and TMR 3
Tier 1 cost-down, no change to the audio path. U9 becomes a Seeed XIAO
RP2040 on header pins (USB-C, TinyUSB MIDI, its 5V pin is VBUS straight
through), PS1 becomes a 2 W unregulated Traco TBA 2-0522 on KiCad's stock
SIP-7 footprint. Rails are now +/-12 V: the +/-15 V TBA 2-0523 would pass
the PGA2310's 16 V absolute maximum at light load. Parts cost drops from
about $145 to about $110.

- gen.py: TBA2_Dual and XIAO_RP2040 symbols, XIAO footprint (Seeed pin
  numbering, USB-C overhang drawn), control sheet rewired to D0-D10,
  power sheet and notes for the unregulated converter, +/-12V rails.
- check.py: new U9 / PS1 pins; NETLIST OK. ERC 0/0.
- Both boards rebuilt and re-routed (Freerouting 1.9), DRC 0 errors; the
  only warnings are jack-nose and USB-C shell silk over the board edge.
- Gerbers, drill, zips, BOM, schematic SVG/PDF and board renders
  regenerated. README and site updated: pin map, power budget
  (~250 mA typical), level budget at +/-12 V, parts list and totals.

Co-Authored-By: Claude Fable 5.1 <noreply@anthropic.com>
Claude-Session: https://claude.ai/code/session_01C8uqpe49go1TPWMsWKKVkn
Connections:
- net +15V renamed +12V
- net -15V renamed -12V
