File: hardware/kicad/power.kicad_sch (KiCad schematic)
At the start: 7 parts

Commit message: Rev C: XIAO RP2040 and Traco TBA 2-0522 replace the Teensy 4.0 and TMR 3
Tier 1 cost-down, no change to the audio path. U9 becomes a Seeed XIAO
RP2040 on header pins (USB-C, TinyUSB MIDI, its 5V pin is VBUS straight
through), PS1 becomes a 2 W unregulated Traco TBA 2-0522 on KiCad's stock
SIP-7 footprint. Rails are now +/-12 V: the +/-15 V TBA 2-0523 would pass
the PGA2310's 16 V absolute maximum at light load. Parts cost drops from
about $145 to about $110.

- gen.py: TBA2_Dual and XIAO_RP2040 symbols, XIAO footprint (Seeed pin
  numbering, USB-C overhang drawn), control sheet rewired to D0-D10,
  power sheet and notes for the unregulated converter, +/-12V rails.
- check.py: new U9 / PS1 pins; NETLIST OK. ERC 0/0.
- Both boards rebuilt and re-routed (Freerouting 1.9), DRC 0 errors; the
  only warnings are jack-nose and USB-C shell silk over the board edge.
- Gerbers, drill, zips, BOM, schematic SVG/PDF and board renders
  regenerated. README and site updated: pin map, power budget
  (~250 mA typical), level budget at +/-12 V, parts list and totals.

Co-Authored-By: Claude Fable 5.1 <noreply@anthropic.com>
Claude-Session: https://claude.ai/code/session_01C8uqpe49go1TPWMsWKKVkn
Parts:
- removed PS1: TMR 3-0523, GhostFader:TRACO_TMR3_SIP8, symbol GhostFader:TMR3_Dual
- added PS1: TBA 2-0522, Converter_DCDC:Converter_DCDC_TRACO_TBA2-xxxx_Dual_THT, symbol GhostFader:TBA2_Dual
Connections:
- net +5V: now also PS1.1 (+Vin)
- net GND: now also PS1.2 (-Vin), PS1.5 (Common)
- net at L1.1: now also PS1.6 (+Vout)
- net at L2.1: now also PS1.4 (-Vout)
- net +15V renamed +12V
- net -15V renamed -12V
- no-connect marks 1 -> 0
Other:
- note added: "Flags (unlabelled) mark +5V, +12V and -12V as driven for ERC, since they sit behind FB1 / L1 / L2."
- note added: "No external power supply. Everything runs from the USB 5 V that the XIAO passes out on its 5V pin (sheet 4). PS1 is a board-mounted isolated 2 W DC-DC module: 5 V in, +/-12 V 80 mA out. Unregulated: the rails follow USB voltage and load, about +/-11 V on a sagging port and up to +/-14 V at 5.25 V and light load; every part on the rails is rated for that (PGA2310 max 16 V). Budget at 5 V: XIAO ~30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"
- note removed: "Flags (unlabelled) mark +5V, +15V and -15V as driven for ERC, since they sit behind FB1 / L1 / L2."
- note removed: "No external power supply. Everything runs from the USB 5 V that the Teensy passes out on VIN (sheet 4). PS1 is a board-mounted isolated DC-DC module: 5 V in, +/-15 V 100 mA out. Remote pin open = on. Budget at 5 V: Teensy 50-100 mA, PS1 ~260 mA for 35 mA per rail, PGA logic + LED 10 mA. ~370 mA typical, 450 mA worst case; USB 2.0 allows 500 mA. All grounds meet once at PS1 Common. Keep PS1 at the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"

Commit message: Rev D: isolate the audio ground from USB
Add a TI ISO7762FDW digital isolator on the four control lines and two
plug-sense lines, a 78L05 that makes +5VA from +12 V for the PGA logic
and the isolator's audio side, and a split ground: GND_USB (XIAO, USB-C,
switch, LED, ferrite, reservoir, DC-DC input) and GND (everything audio).
The two meet only through C45 (1 nF) and R17 (1 M) at PS1. The sense
pull-ups drop from 1 M to 100 k for the isolator's input leakage.

Both boards get two ground pours per layer with a 2 mm copper-free gap
and a rule area that keeps the router out; U8 and PS1 straddle the gap.
The 1590BB board's island is the front-left corner; the narrow board's
is a pocket under the XIAO with the audio ground wrapping beneath it.
ERC 0, netlist checked (61 nets, 263 pins), DRC clean on both routed
boards, and a script check confirms no copper crosses the gap.

README, docs page, schematic exports, renders, gerbers and BOM regenerated.

Co-Authored-By: Claude Fable 5.1 <noreply@anthropic.com>
Claude-Session: https://claude.ai/code/session_013C8baRPktSQjwfdzSRwmAq
Parts:
- added C37, C38: 100n, Capacitor_THT:C_Disc_D5.0mm_W2.5mm_P5.00mm, symbol Device:C
- added C45: 1n 1kV, Capacitor_THT:C_Disc_D5.0mm_W2.5mm_P5.00mm, symbol Device:C
- added R17: 1M, Resistor_THT:R_Axial_DIN0207_L6.3mm_D2.5mm_P10.16mm_Horizontal, symbol Device:R
- added U10: L78L05, Package_TO_SOT_THT:TO-92_Inline_Wide, symbol GhostFader:L78L05
Connections:
- net +12V: now also C37.1, U10.3 (VI)
- net GND: now also C37.2, C38.2, C45.2, R17.2, U10.2 (GND); no longer C11.2, PS1.2 (-Vin)
- new net +5VA: C38.1, U10.1 (VO)
- new net GND_USB: C11.2, C45.1, PS1.2 (-Vin), R17.1
Other:
- note added: "Flags (unlabelled) mark +5V, +12V, -12V and GND_USB as driven for ERC, since they sit behind FB1 / L1 / L2 or the XIAO."
- note added: "Ground barrier. GND_USB (XIAO, USB-C shell, U8 side 1, PS1 input) and GND (everything audio, U8 side 2, PS1 output) meet only here: C45 gives the converter's switching noise a local return so it does not radiate as common mode, R17 stops the audio side floating away when nothing is plugged in. Place both at PS1, on the 2 mm gap in the ground pours. No other copper crosses the gap."
- note added: "No external power supply. Everything runs from the USB 5 V that the XIAO passes out on its 5V pin (sheet 4). PS1 is a board-mounted isolated 2 W DC-DC module: 5 V in, +/-12 V 80 mA out. Unregulated: the rails follow USB voltage and load, about +/-11 V on a sagging port and up to +/-14 V at 5.25 V and light load; every part on the rails is rated for that (PGA2310 max 16 V). Rails: +12 V ~55 mA (an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"
- note added: "U10 78L05: +5VA for the PGA2310 logic, U8 side 2 and the plug-sense pull-ups, about 15 mA. On the audio ground, so the 5 V logic never references USB. Input up to +14 V, 0.15 W in the TO-92."
- note added: "audio star ground"
- note removed: "Flags (unlabelled) mark +5V, +12V and -12V as driven for ERC, since they sit behind FB1 / L1 / L2."
- note removed: "No external power supply. Everything runs from the USB 5 V that the XIAO passes out on its 5V pin (sheet 4). PS1 is a board-mounted isolated 2 W DC-DC module: 5 V in, +/-12 V 80 mA out. Unregulated: the rails follow USB voltage and load, about +/-11 V on a sagging port and up to +/-14 V at 5.25 V and light load; every part on the rails is rated for that (PGA2310 max 16 V). Budget at 5 V: XIAO ~30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"
- note removed: "star ground"
